File: fullOptBattleCartV1.kicad_pcb (KiCad board)
At the start: 2 copper layers, 17 parts, among them M1 Motor_DC, M2 Motor_DC, M3 Motor_DC, M4 Motor_DC, U4 L293D, U5 L293D, U6 LM7905_TO220

Commit message: battlecart modification
Routing:
- added copper zone on B.Cu, net Net-(BT1--)
- added copper zone on F.Cu, net Net-(BT1--)
Other:
- board outline added: 67.9 x 73.7 mm
- board text added: "Design by: Garrett, Fenix, Issac, Alexa Marcus, Levi, Prof. Prater"
- board text added: "fullOptBattleCartV1 RBT353 fall 2024 UAT.edu"
Changed lines of the file:
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@@
     (pad_to_mask_clearance 0)
     (pcbplotparams
-      (layerselection 0x00010fc_ffffffff)
+      (layerselection 0x00010f0_ffffffff)
       (plot_on_all_layers_selection 0x0000000_00000000)
       (disableapertmacros false)
-      (usegerberextensions false)
+      (usegerberextensions true)
       (usegerberattributes true)
       (usegerberadvancedattributes true)
@@
       (psa4output false)
       (plotreference true)
-      (plotvalue true)
+      (plotvalue false)
       (plotinvisibletext false)
       (sketchpadsonfab false)
@@
       (outputformat 1)
       (mirror false)
-      (drillshape 1)
+      (drillshape 0)
       (scaleselection 1)
-      (outputdirectory "")
+      (outputdirectory "gerbers/")
     )
   )
@@
       (stroke (width 0.1) (type solid)) (layer "F.Fab"))
     (pad "" np_thru_hole circle (at -1.6 2 270) (size 1.2 1.2) (drill 1.2) (layers "*.Cu" "*.Mask"))
-    (pad "1" thru_hole roundrect (at 0 0 270) (size 1.7 2) (drill 1) (layers "*.Cu" "*.Mask") (roundrect_rratio 0.147059)
+    (pad "1" thru_hole roundrect (at 0 0 270) (size 1.7 2) (drill 1) (layers "*.Cu" "*.Mask") (roundrect_rratio 0.1470588235)
       (net 3 "Net-(M1-+)") (pinfunction "+") (pintype "passive"))
     (pad "2" thru_hole oval (at 2.5 0 270) (size 1.7 2) (drill 1) (layers "*.Cu" "*.Mask")
@@
     (property "Sheetname" "")
     (attr through_hole)
-    (fp_text reference "U1" (at 0 -27.94 unlocked) (layer "F.SilkS")
+    (fp_text reference "U1" (at 0 -23.495 unlocked) (layer "F.SilkS")
         (effects (font (size 1 1) (thickness 0.1)))
     )
@@
       (stroke (width 0.1) (type solid)) (layer "F.Fab"))
     (pad "" np_thru_hole circle (at -1.6 2 90) (size 1.2 1.2) (drill 1.2) (layers "*.Cu" "*.Mask"))
-    (pad "1" thru_hole roundrect (at 0 0 90) (size 1.7 2) (drill 1) (layers "*.Cu" "*.Mask") (roundrect_rratio 0.147059)
+    (pad "1" thru_hole roundrect (at 0 0 90) (size 1.7 2) (drill 1) (layers "*.Cu" "*.Mask") (roundrect_rratio 0.1470588235)
       (net 9 "Net-(M4-+)") (pinfunction "+") (pintype "passive"))
     (pad "2" thru_hole oval (at 2.5 0 90) (size 1.7 2) (drill 1) (layers "*.Cu" "*.Mask")
@@
     (property "Sheetname" "")
     (attr through_hole)
-    (fp_text reference "U3" (at 10.16 -8.89 unlocked) (layer "F.SilkS")
+    (fp_text reference "U3" (at 0 -4.445 unlocked) (layer "F.SilkS")
         (effects (font (size 1 1) (thickness 0.1)))
     )
@@
     (property "Sheetname" "")
     (attr through_hole)
-    (fp_text reference "U2" (at 10.16 -8.89 180 unlocked) (layer "F.SilkS")
+    (fp_text reference "U2" (at 0 -7.62 unlocked) (layer "F.SilkS")
         (effects (font (size 1 1) (thickness 0.1)))
     )
@@
         (effects (font (size 1 1) (thickness 0.15)))
     )
-    (fp_text user "${REFERENCE}" (at 0 11.43 180 unlocked) (layer "F.Fab")
+    (fp_text user "${REFERENCE}" (at 0 5.715 180 unlocked) (layer "F.Fab")
         (effects (font (size 1 1) (thickness 0.15)))
     )
@@
       (stroke (width 0.1) (type solid)) (layer "F.Fab"))
     (pad "" np_thru_hole circle (at -1.6 2 90) (size 1.2 1.2) (drill 1.2) (layers "*.Cu" "*.Mask"))
-    (pad "1" thru_hole roundrect (at 0 0 90) (size 1.7 2) (drill 1) (layers "*.Cu" "*.Mask") (roundrect_rratio 0.147059)
+    (pad "1" thru_hole roundrect (at 0 0 90) (size 1.7 2) (drill 1) (layers "*.Cu" "*.Mask") (roundrect_rratio 0.1470588235)
       (net 7 "Net-(M3-+)") (pinfunction "+") (pintype "passive"))
     (pad "2" thru_hole oval (at 2.5 0 90) (size 1.7 2) (drill 1) (layers "*.Cu" "*.Mask")
@@
     (fp_line (start 4.95 3.4) (end 4.95 -2.35)
       (stroke (width 0.1) (type solid)) (layer "F.Fab"))
-    (pad "1" thru_hole roundrect (at 0 0) (size 1.7 2) (drill 1) (layers "*.Cu" "*.Mask") (roundrect_rratio 0.147059)
+    (pad "1" thru_hole roundrect (at 0 0) (size 1.7 2) (drill 1) (layers "*.Cu" "*.Mask") (roundrect_rratio 0.1470588235)
       (net 1 "Net-(BT1-+)") (pinfunction "+") (pintype "passive"))
     (pad "2" thru_hole oval (at 2.5 0) (size 1.7 2) (drill 1) (layers "*.Cu" "*.Mask")
@@
       (stroke (width 0.1) (type solid)) (layer "F.Fab"))
     (pad "" np_thru_hole circle (at -1.6 2 270) (size 1.2 1.2) (drill 1.2) (layers "*.Cu" "*.Mask"))
-    (pad "1" thru_hole roundrect (at 0 0 270) (size 1.7 2) (drill 1) (layers "*.Cu" "*.Mask") (roundrect_rratio 0.147059)
+    (pad "1" thru_hole roundrect (at 0 0 270) (size 1.7 2) (drill 1) (layers "*.Cu" "*.Mask") (roundrect_rratio 0.1470588235)
       (net 5 "Net-(M2-+)") (pinfunction "+") (pintype "passive"))
     (pad "2" thru_hole oval (at 2.5 0 270) (size 1.7 2) (drill 1) (layers "*.Cu" "*.Mask")
@@
       (rotate (xyz 0 0 0))
     )
+  )
+  (gr_rect (start 40.64 32.385) (end 108.585 106.045)
+    (stroke (width 0.1) (type default)) (fill none) (layer "Edge.Cuts"))
+  (gr_circle (center 104.775 36.195) (end 107.315 38.1)
+    (stroke (width 0.1) (type default)) (fill none) (layer "Edge.Cuts"))
+  (gr_circle (center 44.45 101.6) (end 46.99 103.505)
+    (stroke (width 0.1) (type default)) (fill none) (layer "Edge.Cuts"))
+  (gr_circle (center 104.775 101.6) (end 107.315 103.505)
+    (stroke (width 0.1) (type default)) (fill none) (layer "Edge.Cuts"))
+  (gr_circle (center 44.45 36.195) (end 46.99 38.1)
+    (stroke (width 0.1) (type default)) (fill none) (layer "Edge.Cuts"))
+  (gr_text "fullOptBattleCartV1\nRBT353 fall 2024\nUAT.edu" (at 107.315 95.885 90) (layer "F.SilkS")
+    (effects (font (size 1 1) (thickness 0.15)) (justify left bottom))
+  )
+  (gr_text "Design by:\nGarrett, Fenix, Issac, Alexa\nMarcus, Levi, Prof. Prater\n" (at 107.315 70.485 90) (layer "F.SilkS")
+    (effects (font (size 1 1) (thickness 0.15)) (justify left bottom))
   )
   (segment (start 70.445 98.385) (end 70.465 98.385) (width 0.25) (layer "F.Cu") (net 1))
@@
   (segment (start 90.17 55.245) (end 88.9 56.515) (width 0.25) (layer "B.Cu") (net 45))
   (segment (start 90.17 44.45) (end 90.17 55.245) (width 0.25) (layer "B.Cu") (net 45))
+  (zone (net 2) (net_name "Net-(BT1--)") (layer "F.Cu") (hatch edge 0.5)
+    (priority 1)
+    (connect_pads (clearance 0.5))
+    (min_thickness 0.25) (filled_areas_thickness no)
+    (fill yes (thermal_gap 0.5) (thermal_bridge_width 0.5))
+    (polygon
+      (pts
+        (xy 39.37 31.115)
+        (xy 110.49 31.115)
+        (xy 110.49 107.315)
+        (xy 39.37 107.315)
+      )
+    )
+  )
+  (zone (net 2) (net_name "Net-(BT1--)") (layer "F.Cu") (hatch edge 0.5)
+    (connect_pads (clearance 0.5))
+    (min_thickness 0.25) (filled_areas_thickness no)
+    (fill yes (thermal_gap 0.5) (thermal_bridge_width 0.5))
+    (polygon
+      (pts
+        (xy 39.37 31.115)
+        (xy 110.49 31.115)
+        (xy 110.49 107.315)
+        (xy 39.37 107.315)
+      )
+    )
+  )
+  (zone (net 2) (net_name "Net-(BT1--)") (layer "B.Cu") (hatch edge 0.5)
+    (priority 2)
+    (connect_pads (clearance 0.5))
+    (min_thickness 0.25) (filled_areas_thickness no)
+    (fill yes (thermal_gap 0.5) (thermal_bridge_width 0.5))
+    (polygon
+      (pts
+        (xy 39.37 31.115)
+        (xy 109.22 31.115)
+        (xy 109.22 107.315)
+        (xy 39.37 107.315)
+      )
+    )
+  )
 )
